File: pcb/keyboard.kicad_pcb (KiCad board)
At the start: 2 copper layers, 435.8 x 140.5 mm, 158 parts, among them U1 Raspberry_Pi_Pico, U2 Raspberry_Pi_Pico

Commit message: forgot to save
Parts:
- added U3: TRRS, ScottoKeebs_Components:TRRS_PJ-320A, F.Cu at (434.9, 182.2)
- added U4: TRRS, ScottoKeebs_Components:TRRS_PJ-320A, F.Cu at (476.2, 129.8)
Connections:
- U1 pad 28: unconnected-(U1-GND-Pad28) -> Net-(U3-SLEEVE)
- U1 pad 31: unconnected-(U1-GPIO26_ADC0-Pad31) -> Net-(U1-GPIO26_ADC0)
- U1 pad 32: unconnected-(U1-GPIO27_ADC1-Pad32) -> Net-(U1-GPIO27_ADC1)
- U1 pad 40: unconnected-(U1-VBUS-Pad40) -> Net-(U1-VBUS)
- U2 pad 28: unconnected-(U2-GND-Pad28) -> Net-(U4-SLEEVE)
- U2 pad 31: unconnected-(U2-GPIO26_ADC0-Pad31) -> Net-(U2-GPIO26_ADC0)
- U2 pad 32: unconnected-(U2-GPIO27_ADC1-Pad32) -> Net-(U2-GPIO27_ADC1)
- U2 pad 40: unconnected-(U2-VBUS-Pad40) -> Net-(U2-VBUS)
Routing:
- net Net-(U2-GPIO26_ADC0): track 0.00 -> 216.0 mm
- net Net-(U2-GPIO27_ADC1): track 0.00 -> 212.0 mm
- net Net-(U4-SLEEVE): track 0.00 -> 209.2 mm
- net Net-(U2-VBUS): track 0.00 -> 200.1 mm
- net R COL3: track 233.8 -> 363.2 mm
- net Net-(U1-VBUS): track 0.00 -> 59.6 mm
- net Net-(U1-GPIO27_ADC1): track 0.00 -> 39.0 mm
- net Net-(U1-GPIO26_ADC0): track 0.00 -> 35.5 mm
- net Net-(U3-SLEEVE): track 0.00 -> 23.0 mm
- net R COL6: track 184.7 -> 183.0 mm
- net unconnected-(U2-GND-Pad38): track 0.00 -> 1.56 mm
- net R COL5: track 197.0 -> 195.7 mm
- net R COL4: track 209.4 -> 208.1 mm
- net R COL7: track 158.3 -> 159.1 mm
- removed copper zone on B.Cu, net GND
- removed copper zone on F.Cu, net GND
Other:
- outline, holes or cut-outs redrawn
