File: pcb/keyboard.kicad_sch (KiCad schematic)
At the start: 160 parts, among them U1 Raspberry_Pi_Pico, U2 Raspberry_Pi_Pico, U3 TRRS, U4 TRRS

Commit message: forgot to save
Connections:
- net at U4.1 (SLEEVE): now also U2.28 (GND); no longer U2.26 (GPIO20)
- net at U4.2 (TIP): now also U2.40 (VBUS); no longer U2.38 (GND)
- net at U4.3 (RING1): now also U2.32 (GPIO27_ADC1); no longer U2.30 (RUN)
- net at U4.4 (RING2): now also U2.31 (GPIO26_ADC0); no longer U2.29 (GPIO22)
Other:
- moved on the sheet: U4
Changed lines of the file:
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@@
 	(wire
 		(pts
-			(xy 298.45 125.73) (xy 308.61 125.73)
-		)
-		(stroke
-			(width 0)
-			(type default)
-		)
-	)
-	(wire
-		(pts
 			(xy 175.26 195.58) (xy 175.26 215.9)
 		)
@@
 	(wire
 		(pts
-			(xy 298.45 118.11) (xy 308.61 118.11)
+			(xy 269.24 256.54) (xy 269.24 276.86)
 		)
 		(stroke
@@
 	(wire
 		(pts
-			(xy 269.24 256.54) (xy 269.24 276.86)
+			(xy 304.8 208.28) (xy 314.96 208.28)
 		)
 		(stroke
@@
 	(wire
 		(pts
-			(xy 304.8 208.28) (xy 314.96 208.28)
+			(xy 175.26 215.9) (xy 175.26 236.22)
 		)
 		(stroke
@@
 	(wire
 		(pts
-			(xy 175.26 215.9) (xy 175.26 236.22)
+			(xy 245.11 228.6) (xy 254 228.6)
 		)
 		(stroke
@@
 	(wire
 		(pts
-			(xy 245.11 228.6) (xy 254 228.6)
+			(xy 298.45 110.49) (xy 312.42 110.49)
 		)
 		(stroke
@@
 	(wire
 		(pts
-			(xy 298.45 95.25) (xy 308.61 95.25)
+			(xy 140.97 228.6) (xy 149.86 228.6)
 		)
 		(stroke
@@
 	(wire
 		(pts
-			(xy 140.97 228.6) (xy 149.86 228.6)
+			(xy 248.92 167.64) (xy 248.92 175.26)
 		)
 		(stroke
@@
 	(wire
 		(pts
-			(xy 248.92 167.64) (xy 248.92 175.26)
+			(xy 179.07 96.52) (xy 189.23 96.52)
 		)
 		(stroke
@@
 	(wire
 		(pts
-			(xy 179.07 96.52) (xy 189.23 96.52)
+			(xy 298.45 113.03) (xy 312.42 113.03)
 		)
 		(stroke
@@
 	(wire
 		(pts
+			(xy 298.45 120.65) (xy 312.42 120.65)
+		)
+		(stroke
+			(width 0)
+			(type default)
+		)
+	)
+	(wire
+		(pts
 			(xy 165.1 175.26) (xy 165.1 195.58)
 		)
@@
 	(wire
 		(pts
-			(xy 298.45 115.57) (xy 308.61 115.57)
-		)
-		(stroke
-			(width 0)
-			(type default)
-		)
-	)
-	(wire
-		(pts
 			(xy 254 208.28) (xy 264.16 208.28)
 		)
@@
 	(wire
 		(pts
-			(xy 308.61 95.25) (xy 308.61 113.03)
+			(xy 312.42 90.17) (xy 312.42 107.95)
 		)
 		(stroke
@@
 	(wire
 		(pts
-			(xy 308.61 125.73) (xy 308.61 120.65)
+			(xy 312.42 115.57) (xy 312.42 120.65)
 		)
 		(stroke
@@
 		)
 	)
+	(wire
+		(pts
+			(xy 312.42 90.17) (xy 298.45 90.17)
+		)
+		(stroke
+			(width 0)
+			(type default)
+		)
+	)
 	(global_label "R COL0"
 		(shape input)
@@
 	(symbol
 		(lib_id "ScottoKeebs:Placeholder_TRRS")
-		(at 317.5 123.19 0)
+		(at 321.31 118.11 0)
 		(unit 1)
 		(exclude_from_sim no)
@@
 		(fields_autoplaced yes)
 		(property "Reference" "U4"
-			(at 323.85 115.5699 0)
+			(at 327.66 110.4899 0)
 			(effects
 				(font
@@
 		)
 		(property "Value" "TRRS"
-			(at 323.85 118.1099 0)
+			(at 327.66 113.0299 0)
 			(effects
 				(font
@@
 		)
 		(property "Footprint" "ScottoKeebs_Components:TRRS_PJ-320A"
-			(at 321.31 123.19 0)
+			(at 325.12 118.11 0)
 			(effects
 				(font
@@
 		)
 		(property "Datasheet" ""
-			(at 321.31 123.19 0)
+			(at 325.12 118.11 0)
 			(effects
 				(font
@@
 		)
 		(property "Description" ""
-			(at 317.5 123.19 0)
+			(at 321.31 118.11 0)
 			(effects
 				(font
